File: projeto 01.sch (KiCad schematic (older format))
At the start: 5 parts

Commit message: Selecionei as Footprints
Parts:
- C1: renamed from C?; footprint (none) -> Capacitor_THT:C_Disc_D3.0mm_W2.0mm_P2.50mm
- R1, R2, R3: renamed from R?; footprint (none) -> Resistor_THT:R_Axial_DIN0204_L3.6mm_D1.6mm_P7.62mm_Horizontal
- gave numbers to parts that had none: 1
Changed lines of the file:
@@
 $EndDescr
 $Comp
-L Device:R_Small R?
+L Device:R_Small R2
 U 1 1 5D4DF63A
 P 6000 3650
-F 0 "R?" H 6050 3700 50  0000 L CNN
+F 0 "R2" H 6050 3700 50  0000 L CNN
 F 1 "510k" H 6059 3605 50  0000 L CNN
-F 2 "" H 6000 3650 50  0001 C CNN
+F 2 "Resistor_THT:R_Axial_DIN0204_L3.6mm_D1.6mm_P7.62mm_Horizontal" H 6000 3650 50  0001 C CNN
 F 3 "~" H 6000 3650 50  0001 C CNN
 	1    6000 3650
@@
 $EndComp
 $Comp
-L Device:R_Small R?
+L Device:R_Small R1
 U 1 1 5D4E1E08
 P 5800 3400
-F 0 "R?" V 5950 3350 50  0000 L CNN
+F 0 "R1" V 5950 3350 50  0000 L CNN
 F 1 "1k" V 5859 3355 50  0000 L CNN
-F 2 "" H 5800 3400 50  0001 C CNN
+F 2 "Resistor_THT:R_Axial_DIN0204_L3.6mm_D1.6mm_P7.62mm_Horizontal" H 5800 3400 50  0001 C CNN
 F 3 "~" H 5800 3400 50  0001 C CNN
 	1    5800 3400
@@
 $EndComp
 $Comp
-L Device:C_Small C?
+L Device:C_Small C1
 U 1 1 5D4E2E7F
 P 5450 3400
-F 0 "C?" V 5221 3400 50  0000 C CNN
+F 0 "C1" V 5221 3400 50  0000 C CNN
 F 1 "20nF" V 5312 3400 50  0000 C CNN
-F 2 "" H 5450 3400 50  0001 C CNN
+F 2 "Capacitor_THT:C_Disc_D3.0mm_W2.0mm_P2.50mm" H 5450 3400 50  0001 C CNN
 F 3 "~" H 5450 3400 50  0001 C CNN
 	1    5450 3400
@@
 $EndComp
 $Comp
-L Transistor_BJT:BC548 Q?
+L Transistor_BJT:BC548 Q1
 U 1 1 5D4E3938
 P 6300 3400
-F 0 "Q?" H 6491 3446 50  0000 L CNN
+F 0 "Q1" H 6491 3446 50  0000 L CNN
 F 1 "BC548" H 6491 3355 50  0000 L CNN
 F 2 "Package_TO_SOT_THT:TO-92_Inline" H 6500 3325 50  0001 L CIN
@@
 $EndComp
 $Comp
-L Device:R_Small R?
+L Device:R_Small R3
 U 1 1 5D4E45DE
 P 6400 3800
-F 0 "R?" H 6450 3850 50  0000 L CNN
+F 0 "R3" H 6450 3850 50  0000 L CNN
 F 1 "10k" H 6459 3755 50  0000 L CNN
-F 2 "" H 6400 3800 50  0001 C CNN
+F 2 "Resistor_THT:R_Axial_DIN0204_L3.6mm_D1.6mm_P7.62mm_Horizontal" H 6400 3800 50  0001 C CNN
 F 3 "~" H 6400 3800 50  0001 C CNN
 	1    6400 3800
@@
 $EndComp
 $Comp
-L power:GND #PWR?
+L power:GND #PWR0101
 U 1 1 5D4E527A
 P 6400 4100
-F 0 "#PWR?" H 6400 3850 50  0001 C CNN
+F 0 "#PWR0101" H 6400 3850 50  0001 C CNN
 F 1 "GND" H 6405 3927 50  0000 C CNN
 F 2 "" H 6400 4100 50  0001 C CNN
@@
 $EndComp
 $Comp
-L power:VCC #PWR?
+L power:VCC #PWR0102
 U 1 1 5D4E5B86
 P 6400 3000
-F 0 "#PWR?" H 6400 2850 50  0001 C CNN
+F 0 "#PWR0102" H 6400 2850 50  0001 C CNN
 F 1 "VCC" H 6417 3173 50  0000 C CNN
 F 2 "" H 6400 3000 50  0001 C CNN
@@
 	6400 3900 6400 4100
 $Comp
-L power:GND #PWR?
+L power:GND #PWR0103
 U 1 1 5D4E726A
 P 6000 3950
-F 0 "#PWR?" H 6000 3700 50  0001 C CNN
+F 0 "#PWR0103" H 6000 3700 50  0001 C CNN
 F 1 "GND" H 6005 3777 50  0000 C CNN
 F 2 "" H 6000 3950 50  0001 C CNN
